File: ECAD/StrikeDetector/StrikeDetector.sch (EAGLE design)
At the start: 32 parts, among them J1 10118193-0001LF, U1 MMBT2222A-7-F, U2 MMBT2222A-7-F, U3 LSM9DS1TR, U4 ESP32-WROOM-32, U6 AP2112K-3.3TRG1

Commit message: Updated PCB Design
Parts:
- added JP3: (no value), microbuilder:HEADER-1X6ROUND
- added R11: 100kΩ, microbuilder:RESISTOR0603
- added SW1, SW2: KMR211GLFS, adafruit:SPST_TACT-KMR2
Connections:
- new net N$13: JP3.2
- new net N$17: JP3.6
- net 3.3V: now also R11.2
- net GND: now also JP3.1, SW1.P, SW1.P1, SW2.P, SW2.P1
- net GPIO0: now also SW2.S, SW2.S1
- net RESET: now also R11.1, SW1.S, SW1.S1
- net RXD0: now also JP3.4
- net TXD0: now also JP3.5
- net VIN: now also JP3.3
