File: ECAD/StrikeDetector/StrikeDetector.brd (EAGLE design)
At the start: 24 x 48 mm, 36 parts, among them J1 10118193-0001LF, SW1 KMR211GLFS, SW2 KMR211GLFS, U1 MMBT2222A-7-F, U2 MMBT2222A-7-F, U3 LSM9DS1TR, U4 ESP32-WROOM-32, U5 CP2104-F03-GM, U6 AP2112K-3.3TRG1

Commit message: Updated ECAD
Added Pull up resistors for the pins I was missing
Parts:
- added R12, R13, R14, R15, R16: 10kΩ, microbuilder:0603
- R6, R7: value 4.7kΩ -> 10kΩ
- moved R6 0.80 mm to (14.8, 21.2)
- moved R7 0.70 mm to (16.4, 21.3)
- moved C1 0.22 mm to (11.4, 20.3)
- moved C2 0.22 mm to (13.0, 20.3)
Connections:
- new net N$12: R12.1, U3.7
- new net N$14: R13.1, U3.13
- new net N$15: R14.1, U3.8
- new net N$16: R15.1, U3.5
- new net N$18: R16.1, U3.6
- net 3.3V: now also R12.2, R13.2, R14.2, R15.2, R16.2
Routing:
- net 3.3V: track 70.7 -> 89.8 mm
- net N$12: track 0.00 -> 6.94 mm
- net N$14: track 0.00 -> 6.57 mm
- net N$15: track 0.00 -> 4.70 mm
- net N$16: track 0.00 -> 2.05 mm
- net N$18: track 0.00 -> 1.90 mm
- net SCL: track 28.3 -> 29.5 mm
- net SDA: track 29.2 -> 29.7 mm
